File: pcb/power-module.kicad_pcb (KiCad board)
At the start: 4 copper layers, 55 x 55 mm, 53 parts, among them J1 USB_C_PowerOnly_6P, J2 Power, U1 AZ1084-3.3, U2 LM66200DRLR

Commit message: revamped using different examples
Other:
- board text added: "${COMMIT}"
Changed lines of the file:
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@@
+		)
+	)
+	(gr_text "${COMMIT}"
+		(at 77 150 0)
+		(layer "B.SilkS")
+		(effects
+			(font
+				(size 1.27 1.27)
+				(thickness 0.127)
+				(bold yes)
+			)
 		)
 	)

Commit message: optimized script; still fighting some errors
Other:
- board text added: "<<hash>>"
- board text removed: "${COMMIT}"
Changed lines of the file:
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@@
 		)
 	)
-	(gr_text "${COMMIT}"
+	(gr_text "<<hash>>"
 		(at 77 150 0)
 		(layer "B.SilkS")
