File: pcb/power-module.kicad_pcb (KiCad board)
At the start: 4 copper layers, 55 x 55 mm, 51 parts, among them J1 USB_C_PowerOnly_6P, J2 Power, U1 AZ1084-3.3, U2 LM66200DRLR

Commit message: Minor clean up and dimensioning
Parts:
- R4: value 1k -> 4.7k
- moved LOGO4 1.47 mm to (99.0, 149.5)
- moved kibuzzard-681CF78D 1.47 mm to (99.1, 151.1)
Routing:
- net GND: vias 90 -> 100

Commit message: Updated mounting hole footprint and dimensions
Other:
- board text added: "x 6"
Changed lines of the file:
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@@
 		(sheetname "/")
 		(sheetfile "power-module.kicad_sch")
-		(clearance 1)
 		(attr exclude_from_bom)
 		(fp_circle
 			(center 0 0)
+			(end 1.6 0)
+			(stroke
+				(width 0.15)
+				(type solid)
+			)
+			(fill no)
+			(layer "Cmts.User")
+		)
+		(fp_circle
+			(center 0 0)
 			(end 3.2 0)
 			(stroke
@@
 		(fp_circle
 			(center 0 0)
+			(end 1.6 0)
+			(stroke
+				(width 0.15)
+				(type solid)
+			)
+			(fill no)
+			(layer "Cmts.User")
+		)
+		(fp_circle
+			(center 0 0)
 			(end 3.2 0)
 			(stroke
@@
 		(sheetname "/")
 		(sheetfile "power-module.kicad_sch")
-		(clearance 1)
 		(attr exclude_from_bom)
 		(fp_circle
 			(center 0 0)
+			(end 1.6 0)
+			(stroke
+				(width 0.15)
+				(type solid)
+			)
+			(fill no)
+			(layer "Cmts.User")
+		)
+		(fp_circle
+			(center 0 0)
 			(end 3.2 0)
 			(stroke
@@
 		(sheetname "/")
 		(sheetfile "power-module.kicad_sch")
-		(clearance 1)
 		(attr exclude_from_bom)
 		(fp_circle
 			(center 0 0)
+			(end 1.6 0)
+			(stroke
+				(width 0.15)
+				(type solid)
+			)
+			(fill no)
+			(layer "Cmts.User")
+		)
+		(fp_circle
+			(center 0 0)
 			(end 3.2 0)
 			(stroke
@@
 		(sheetname "/")
 		(sheetfile "power-module.kicad_sch")
-		(clearance 1)
 		(attr exclude_from_bom)
 		(fp_circle
 			(center 0 0)
+			(end 1.6 0)
+			(stroke
+				(width 0.15)
+				(type solid)
+			)
+			(fill no)
+			(layer "Cmts.User")
+		)
+		(fp_circle
+			(center 0 0)
 			(end 3.2 0)
 			(stroke
@@
 		(fp_circle
 			(center 0 0)
+			(end 1.6 0)
+			(stroke
+				(width 0.15)
+				(type solid)
+			)
+			(fill no)
+			(layer "Cmts.User")
+		)
+		(fp_circle
+			(center 0 0)
 			(end 3.2 0)
 			(stroke
@@
 		)
 	)
+	(gr_text "x 6"
+		(at 118.8 167.9 0)
+		(layer "Dwgs.User")
+		(effects
+			(font
+				(size 1 1)
+				(thickness 0.15)
+			)
+			(justify left bottom)
+		)
+	)
+	(gr_text "x 6"
+		(at 119.9 169.9 0)
+		(layer "Dwgs.User")
+		(effects
+			(font
+				(size 1 1)
+				(thickness 0.15)
+			)
+			(justify left bottom)
+		)
+	)
 	(gr_text "Score Line"
 		(at 32 110 0)
@@
 			(units 3)
 			(units_format 0)
-			(precision 4)
+			(precision 2)
 			(override_value "3.0")
-			(suppress_zeroes yes)
 		)
 		(style
@@
 			(units 3)
 			(units_format 0)
-			(precision 4)
-			(override_value "1.6")
-			(suppress_zeroes yes)
+			(precision 2)
+			(override_value "1.60")
 		)
 		(style
@@
 			(keep_text_aligned yes)
 		)
-		(gr_text "R 1.6"
+		(gr_text "R 1.60"
 			(at 115.508114 167.412191 0)
 			(layer "Dwgs.User")
@@
 	)
 	(dimension
+		(type radial)
+		(layer "Dwgs.User")
+		(pts
+			(xy 101 161) (xy 102.066661 164.016991)
+		)
+		(leader_length 5.789665)
+		(format
+			(prefix "R ")
+			(suffix "")
+			(units 3)
+			(units_format 0)
+			(precision 2)
+		)
+		(style
+			(thickness 0.1)
+			(arrow_length 1.27)
+			(text_position_mode 0)
+			(extension_offset 0.5)
+			(keep_text_aligned yes)
+		)
+		(gr_text "R 3.20"
+			(at 116.696539 169.475543 0)
+			(layer "Dwgs.User")
+			(effects
+				(font
+					(size 1 1)
+					(thickness 0.15)
+				)
+			)
+		)
+	)
+	(dimension
 		(type orthogonal)
 		(layer "Dwgs.User")
@@
 			(units 3)
 			(units_format 0)
-			(precision 4)
-			(suppress_zeroes yes)
+			(precision 2)
 		)
 		(style
 			(thickness 0.1)
 			(arrow_length 1.27)
-			(text_position_mode 0)
+			(text_position_mode 2)
 			(arrow_direction outward)
 			(extension_height 0.58642)
@@
 			(keep_text_aligned yes)
 		)
-		(gr_text "4"
-			(at 52 170.25 0)
+		(gr_text "4.00"
+			(at 52 173.2 0)
 			(layer "Dwgs.User")
 			(effects
@@
 			(units 3)
 			(units_format 0)
-			(precision 4)
-			(suppress_zeroes yes)
+			(precision 2)
 		)
 		(style
@@
 			(keep_text_aligned yes)
 		)
-		(gr_text "47"
+		(gr_text "47.00"
 			(at 42.1 137.5 90)
 			(layer "Dwgs.User")
@@
 			(units 3)
 			(units_format 0)
-			(precision 4)
-			(suppress_zeroes yes)
+			(precision 2)
 		)
 		(style
@@
 			(keep_text_aligned yes)
 		)
-		(gr_text "18.2"
+		(gr_text "18.20"
 			(at 74.6 166.65 0)
 			(layer "Dwgs.User")
@@
 			(units 3)
 			(units_format 0)
-			(precision 4)
-			(suppress_zeroes yes)
+			(precision 2)
 		)
 		(style
@@
 			(keep_text_aligned yes)
 		)
-		(gr_text "11.5"
+		(gr_text "11.50"
 			(at 59.75 166.65 0)
 			(layer "Dwgs.User")
@@
 			(units 3)
 			(units_format 0)
-			(precision 4)
-			(suppress_zeroes yes)
+			(precision 2)
 		)
 		(style
@@
 			(keep_text_aligned yes)
 		)
-		(gr_text "55"
+		(gr_text "55.00"
 			(at 114.35 137.5 90)
 			(layer "Dwgs.User")
@@
 			(units 3)
 			(units_format 0)
-			(precision 4)
-			(suppress_zeroes yes)
+			(precision 2)
 		)
 		(style
@@
 			(keep_text_aligned yes)
 		)
-		(gr_text "47"
+		(gr_text "47.00"
 			(at 77.5 102.85 0)
 			(layer "Dwgs.User")
@@
 			(units 3)
 			(units_format 0)
-			(precision 4)
-			(suppress_zeroes yes)
+			(precision 2)
 		)
 		(style
@@
 			(keep_text_aligned yes)
 		)
-		(gr_text "14"
+		(gr_text "14.00"
 			(at 61 106.35 0)
 			(layer "Dwgs.User")
@@
 			(units 3)
 			(units_format 0)
-			(precision 4)
-			(suppress_zeroes yes)
+			(precision 2)
 		)
 		(style
 			(thickness 0.1)
 			(arrow_length 1.27)
-			(text_position_mode 0)
+			(text_position_mode 2)
 			(arrow_direction outward)
 			(extension_height 0.58642)
@@
 			(keep_text_aligned yes)
 		)
-		(gr_text "4"
-			(at 42.1 163 90)
+		(gr_text "4.00"
+			(at 41.4 163 90)
 			(layer "Dwgs.User")
 			(effects
@@
 			(units 3)
 			(units_format 0)
-			(precision 4)
-			(suppress_zeroes yes)
+			(precision 2)
 		)
 		(style
@@
 			(keep_text_aligned yes)
 		)
-		(gr_text "47"
+		(gr_text "47.00"
 			(at 77.5 170.25 0)
 			(layer "Dwgs.User")
@@
 			(units 3)
 			(units_format 0)
-			(precision 4)
-			(suppress_zeroes yes)
+			(precision 2)
 		)
 		(style
@@
 			(keep_text_aligned yes)
 		)
-		(gr_text "20"
+		(gr_text "20.00"
 			(at 78 106.35 0)
 			(layer "Dwgs.User")
@@
 			(units 3)
 			(units_format 0)
-			(precision 4)
-			(suppress_zeroes yes)
+			(precision 2)
 		)
 		(style
@@
 			(keep_text_aligned yes)
 		)
-		(gr_text "55"
+		(gr_text "55.00"
 			(at 77.5 100.15 0)
 			(layer "Dwgs.User")
@@
 			(units 3)
 			(units_format 0)
-			(precision 4)
-			(suppress_zeroes yes)
+			(precision 2)
 		)
 		(style
@@
 			(keep_text_aligned yes)
 		)
-		(gr_text "47"
+		(gr_text "47.00"
 			(at 109.35 137.5 90)
 			(layer "Dwgs.User")
